File: K_Pennywhistle.kicad_sch (KiCad schematic)
At the start: 67 parts, among them J1 Bias Control, J2 Conn_Coaxial, J3 P IN, J4 Conn_Coaxial, Q1 RD15HVF1, Q2 RD15HVF1, Q3 ZVP2106G, T1 BN43-302, T2 TLT BN43-202, T3 Output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

Commit message: first routed draft, fix some errors
Parts:
- D1, D2: footprint (none) -> Diode_SMD:D_0805_2012Metric
Connections:
- net GND: no longer C15.2, C24.2
- net at C10.1, C12.1, C13.1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: no longer T2.1, T2.4
- net at Q3.3 (S), R19.2: now also C22.1, C25.1, L4.1
- net at C11.1, Q2.3 (D), T2.3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: now also C15.2
- net at R12.1, R13.1, R15.2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: now also C14.2
- net at C18.1, C19.1, R15.1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: no longer C14.2
- new net: T2.1, T2.4
- now unconnected: C24.1
Other:
- moved on the sheet: C1, C15, C2, C22, C23, C25, C26, C3, C4, D2, J1, J3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

Commit message: near RTM, iBom and 3D image added
Parts:
- added H105, H106, H107, H108: MountingHole_Pad, MountingHole:MountingHole_3.2mm_M3_ISO14580_Pad_TopBottom, symbol Mechanical:MountingHole_Pad
- C1, C14, C17, C18, C22, C23, C24, C26, C3, C4, C7, C9: footprint Capacitor_SMD:C_0805_2012Metric_Pad1.18x1.45mm_HandSolder -> Capacitor_SMD:C_1206_3216Metric_Pad1.33x1.80mm_HandSolder
- C10, C11, C12, C13, C16, C51, C6: footprint Capacitor_SMD:C_1812_4532Metric_Pad1.57x3.40mm_HandSolder -> Capacitor_SMD:C_1206_3216Metric_Pad1.33x1.80mm_HandSolder
- J2: value Conn_Coaxial -> DMZ
- J4: value Conn_Coaxial -> SMA
Connections:
- net +12V: now also C26.1, L3.2
- net GND: now also C24.2, H105.1, H106.1, H107.1, H108.1
- net at C10.1, C12.1, C13.1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: now also T2.1; no longer C26.1, L3.2
- net at C22.1, C25.1, L4.1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: now also C24.1
- net at T2.1: no longer T2.4
Other:
- moved on the sheet: C24

Commit message: minor mods, new Gerber & iBom, schematic pdf,RTM
Other:
- note added: "1/1"
- note added: "14/05/2026"
- note added: "Pennywhistle KE9H OpenHPSDR HF Amplifier"
Changed lines of the file:
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@@
 	(generator_version "10.0")
 	(paper "A4")
+	(text "14/05/2026"
+		(exclude_from_sim no)
+		(at 213.36 193.04 0)
+		(effects
+			(font
+				(size 1.27 1.27)
+			)
+		)
+	)
 	(text "2T\n"
 		(exclude_from_sim no)
@@
 			(font
 				(size 1.27 1.27)
+			)
+		)
+	)
+	(text "Pennywhistle\n\nKE9H OpenHPSDR HF Amplifier"
+		(exclude_from_sim no)
+		(at 229.87 173.99 0)
+		(effects
+			(font
+				(size 2.54 2.54)
+				(thickness 0.3048)
+				(bold yes)
+				(color 53 51 255 1)
 			)
 		)
@@
 			)
 		)
+	)
+	(text "1/1"
+		(exclude_from_sim no)
+		(at 189.23 184.15 0)
+		(effects
+			(font
+				(size 1.27 1.27)
+				(thickness 0.254)
+				(bold yes)
+			)
+		)
